File: SensorBoard/SensorBoard.sch (KiCad schematic (older format))
At the start: 16 parts, among them U1 PHOTODIODE, U2 PHOTODIODE

Commit message: moving a resistor to the wrong place.
Please undo me!
Parts:
- C1, C2: symbol C -> C-RESCUE-SensorBoard
- R1, R2, R3, R4: symbol R -> R-RESCUE-SensorBoard
Connections:
- net at OPAMP2.7 (Vdd), PHOTODIODE_OUT1.2 (PM): no longer R4.2
- net at OPAMP2.6 (Vout), U2.~ (V-): no longer R4.1
Other:
- moved on the sheet: R4
Changed lines of the file:
@@
 EESchema Schematic File Version 2
+LIBS:SensorBoard-rescue
 LIBS:power
 LIBS:device
@@
 LIBS:memory
 LIBS:xilinx
-LIBS:special
 LIBS:microcontrollers
 LIBS:dsp
@@
 LIBS:HMC1051
 LIBS:SensorBoard-cache
-EELAYER 27 0
+EELAYER 25 0
 EELAYER END
 $Descr A4 11693 8268
@@
 $EndComp
 $Comp
-L C C2
+L C-RESCUE-SensorBoard C2
 U 1 1 5552AD2C
 P 6350 7050
@@
 $EndComp
 $Comp
-L C C1
+L C-RESCUE-SensorBoard C1
 U 1 1 5552AD39
 P 3000 6100
@@
 $EndComp
 $Comp
-L R R1
+L R-RESCUE-SensorBoard R1
 U 1 1 5552AD43
 P 3050 6500
@@
 $EndComp
 $Comp
-L R R3
+L R-RESCUE-SensorBoard R3
 U 1 1 5552AD50
 P 6350 7400
@@
 $EndComp
 $Comp
-L R R4
+L R-RESCUE-SensorBoard R4
 U 1 1 5552AD56
-P 8250 6600
-F 0 "R4" V 8330 6600 40  0000 C CNN
-F 1 "0.3" V 8257 6601 40  0000 C CNN
-F 2 "~" V 8180 6600 30  0000 C CNN
-F 3 "~" H 8250 6600 30  0000 C CNN
-	1    8250 6600
+P 7950 6200
+F 0 "R4" V 8030 6200 40  0000 C CNN
+F 1 "0.3" V 7957 6201 40  0000 C CNN
+F 2 "~" V 7880 6200 30  0000 C CNN
+F 3 "~" H 7950 6200 30  0000 C CNN
+	1    7950 6200
 	0    -1   -1   0
 $EndComp
 $Comp
-L R R2
+L R-RESCUE-SensorBoard R2
 U 1 1 5552AD5C
 P 4350 5350
